File: boards/field_device/humidity_sensor.kicad_sch (KiCad schematic)
At the start: 3 parts, among them U1 CHT20MEMS

Commit message: connected crystal
Connections:
- no-connect marks 0 -> 2
Changed lines of the file:
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@@
 		(color 0 0 0 0)
+	)
+	(no_connect
+		(at 41.91 22.86)
+	)
+	(no_connect
+		(at 59.69 22.86)
 	)
 	(wire
