File: boards/field_device/humidity_sensor.kicad_sch (KiCad schematic)
At the start: 3 parts, among them U1 CHT20MEMS

Commit message: rev 5?
Parts:
- C1: value 10uF -> 10u
Connections:
- net VDD: now reaches R1.2, U1.2 (VDD)
Other:
- title: (none) -> Field Device Humidity Sensor
Changed lines of the file:
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@@
 	(generator_version "10.0")
 	(paper "A4")
+	(title_block
+		(title "Field Device Humidity Sensor")
+		(date "2026-10-09")
+		(rev "5")
+	)
 	(junction
 		(at 34.29 25.4)
@@
 			(width 0)
 			(type default)
+		)
+	)
+	(label "VDD"
+		(at 40.64 25.4 180)
+		(effects
+			(font
+				(size 1.27 1.27)
+			)
+			(justify right bottom)
 		)
 	)
@@
 			)
 		)
-		(property "Value" "10uF"
+		(property "Value" "10u"
 			(at 25.4 30.4799 0)
 			(show_name no)

Commit message: change components to fit manufacturing capability
Parts:
- C1: value 10u -> 10uF
Changed lines of the file:
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@@
 			)
 		)
-		(property "Value" "10u"
+		(property "Value" "10uF"
 			(at 25.4 30.4799 0)
 			(show_name no)

Commit message: idk atp
Parts:
- C1: value 10uF -> CL10A106KP8NNNC 10uF
- R1: value 330R -> 0603WAF3300T5E 330R; footprint Resistor_SMD:R_0402_1005Metric_Pad0.72x0.64mm_HandSolder -> Capacitor_SMD:C_0603_1608Metric
Changed lines of the file:
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@@
 			)
 		)
-		(property "Value" "330R"
+		(property "Value" "0603WAF3300T5E 330R"
 			(at 26.67 21.59 90)
 			(show_name no)
@@
 			)
 		)
-		(property "Footprint" "Resistor_SMD:R_0402_1005Metric_Pad0.72x0.64mm_HandSolder"
+		(property "Footprint" "Capacitor_SMD:C_0603_1608Metric"
 			(at 26.67 27.178 90)
 			(hide yes)
@@
 			)
 		)
-		(property "Value" "10uF"
+		(property "Value" "CL10A106KP8NNNC 10uF"
 			(at 25.4 30.4799 0)
 			(show_name no)
