File: boards/field_device/lora_module.kicad_sch (KiCad schematic)
At the start: 1 part, among them U6 SX1262IMLTRT

Commit message: RF is fun!
Parts:
- added AE1: Antenna, Package_DFN_QFN:DFN-8-1EP_2x3mm_P0.5mm_EP0.61x2.2mm, symbol Device:Antenna
- added C15: 10uF, symbol Device:C
- added C16, C17, C18: 100nF, symbol Device:C
- added C19: 470nF, symbol Device:C
- added C20: 47nF, symbol Device:C
- added C21, C22: 100pF, symbol Device:C
- added C23: C_Shunt_1, symbol Device:C
- added C24: C_Shunt_2, symbol Device:C
- added L2: 47nH, symbol Device:L
- added L3: L_Series, symbol Device:L
- added Y1: Crystal, Crystal:Crystal_SMD_3225-4Pin_3.2x2.5mm, symbol Device:Crystal
Connections:
- net VDD_RADIO: now reaches U6.1 (VDD_IN)
- net VDD_RADIO: now also C18.1
- net +3.3V: now reaches U6.10 (VBAT)
- net +3.3V: now also U6.11 (VBAT_IO), C15.1, C16.1, C17.1
- net GND: now reaches U6.2 (GND)
- net GND: now also U6.20 (GND), U6.21 (RFI_P), U6.22 (RFI_N), U6.25 (GND), U6.5 (GND), U6.8 (GND), U6.9 (DCC_SW), C15.2, C16.2, C17.2, C18.2, C19.2, C20.2, C21.2, C23.2, C24.2
- net at U6.23 (RFO): now also C22.2, L2.2
- net at U6.24 (VR_PA): now also C20.1, C21.1, L2.1
- net at U6.7 (VREG): now also C19.1
- new net: C22.1, C23.1, L3.1
- new net: AE1.1 (A), C24.1, L3.2
Other:
- note added: "DC block"
- note added: "Matching Network"
- note added: "pull up"

Commit message: connected crystal
Parts:
- removed Y1: Crystal, Crystal:Crystal_SMD_3225-4Pin_3.2x2.5mm, symbol Device:Crystal
- added Y1: Crystal_GND24, Crystal:Crystal_SMD_3225-4Pin_3.2x2.5mm, symbol Device:Crystal_GND24
Connections:
- net GND: now also Y1.2 (G), Y1.4 (G)
- net XTA: now reaches U6.3 (XTA)
- net XTA: now also Y1.3
- net XTB: now reaches U6.4 (XTB)
- net XTB: now also Y1.1
- no-connect marks 0 -> 2
Other:
- note added: "Crystal"
- moved on the sheet: AE1, C15, C16, C17, C18, C19, C20, C21, C22, C23, C24, L2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
