File: boards/field_device/lora_module.kicad_sch (KiCad schematic)
At the start: 15 parts, among them U6 SX1262IMLTRT, Y1 Crystal_GND24

Commit message: connected lora to mcu
Parts:
- U6: footprint UnEasy-LCSC:QFN-24_L4.0-W4.0-P0.50-BL-EP2.6 -> Package_DFN_QFN:QFN-24-1EP_4x4mm_P0.5mm_EP2.15x2.15mm
Connections:
- net DIO1: now reaches U6.13 (DIO1)
- net BUSY: now reaches U6.14 (BUSY)
- net NRST: now reaches U6.15 (NRESET)
- net MISO: now reaches U6.16 (MISO)
- net MOSI: now reaches U6.17 (MOSI)
- net SCK: now reaches U6.18 (SCK)
- net NSS: now reaches U6.19 (NSS)
Changed lines of the file:
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@@
+		)
+	)
+	(hierarchical_label "MISO"
+		(shape output)
+		(at 129.54 55.88 0)
+		(effects
+			(font
+				(size 1.27 1.27)
+			)
+			(justify left)
+		)
+	)
+	(hierarchical_label "NRST"
+		(shape input)
+		(at 129.54 58.42 0)
+		(effects
+			(font
+				(size 1.27 1.27)
+			)
+			(justify left)
+		)
+	)
+	(hierarchical_label "BUSY"
+		(shape output)
+		(at 129.54 60.96 0)
+		(effects
+			(font
+				(size 1.27 1.27)
+			)
+			(justify left)
+		)
+	)
+	(hierarchical_label "MOSI"
+		(shape input)
+		(at 129.54 53.34 0)
+		(effects
+			(font
+				(size 1.27 1.27)
+			)
+			(justify left)
+		)
+	)
+	(hierarchical_label "NSS"
+		(shape input)
+		(at 129.54 48.26 0)
+		(effects
+			(font
+				(size 1.27 1.27)
+			)
+			(justify left)
+		)
+	)
+	(hierarchical_label "SCK"
+		(shape input)
+		(at 129.54 50.8 0)
+		(effects
+			(font
+				(size 1.27 1.27)
+			)
+			(justify left)
+		)
+	)
+	(hierarchical_label "DIO1"
+		(shape output)
+		(at 129.54 63.5 0)
+		(effects
+			(font
+				(size 1.27 1.27)
+			)
+			(justify left)
 		)
 	)
@@
 			)
 		)
-		(property "Footprint" "UnEasy-LCSC:QFN-24_L4.0-W4.0-P0.50-BL-EP2.6"
+		(property "Footprint" "Package_DFN_QFN:QFN-24-1EP_4x4mm_P0.5mm_EP2.15x2.15mm"
 			(at 111.76 67.31 0)
 			(hide yes)

Commit message: fun
Parts:
- C16: renamed from C19; footprint (none) -> Capacitor_SMD:C_0603_1608Metric
- C17: renamed from C15; footprint (none) -> Capacitor_SMD:C_0603_1608Metric
- C18: renamed from C16; footprint (none) -> Capacitor_SMD:C_0603_1608Metric
- C19: renamed from C17; footprint (none) -> Capacitor_SMD:C_0603_1608Metric
- C20: renamed from C18; footprint (none) -> Capacitor_SMD:C_0603_1608Metric
- C21: renamed from C20; footprint (none) -> Capacitor_SMD:C_0603_1608Metric
- C22: renamed from C21; footprint (none) -> Capacitor_SMD:C_0603_1608Metric
- C23: renamed from C22; footprint (none) -> Capacitor_SMD:C_0603_1608Metric
- C24: renamed from C23; footprint (none) -> Capacitor_SMD:C_0603_1608Metric
- C25: renamed from C24; footprint (none) -> Capacitor_SMD:C_0603_1608Metric
- L2, L3: footprint (none) -> Inductor_SMD:L_0603_1608Metric

Commit message: reorganized mcu
Connections:
- net VDD_RADIO is gone; now on net +3.3V: C20.1, U6.1 (VDD_IN)
Other:
- moved on the sheet: C16, C17, C18, C19, C20, Y1

Commit message: added satus leds
Parts:
- renumbered C17 to C14, C18 to C15, C19 to C16, C20 to C17, C16 to C18, C21 to C19, C22 to C20, C23 to C21, C24 to C22, C25 to C23
Changed lines of the file:
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@@
 		(dnp no)
 		(fields_autoplaced yes)
-		(property "Reference" "#PWR042"
+		(property "Reference" "#PWR043"
 			(at 87.63 55.88 0)
 			(hide yes)
@@
 			(project "field_device"
 				(path "/99623870-118f-49fe-bbf0-fb0b890db442/d15b20d6-817c-48cf-abc4-788b93984e6d"
-					(reference "#PWR042")
+					(reference "#PWR043")
 					(unit 1)
 				)
@@
 		(dnp no)
 		(fields_autoplaced yes)
-		(property "Reference" "#PWR034"
+		(property "Reference" "#PWR036"
 			(at -1.27 50.8 0)
 			(hide yes)
@@
 			(project "field_device"
 				(path "/99623870-118f-49fe-bbf0-fb0b890db442/d15b20d6-817c-48cf-abc4-788b93984e6d"
-					(reference "#PWR034")
+					(reference "#PWR036")
 					(unit 1)
 				)
@@
 		(dnp no)
 		(fields_autoplaced yes)
-		(property "Reference" "#PWR041"
+		(property "Reference" "#PWR042"
 			(at 87.63 53.34 0)
 			(hide yes)
@@
 			(project "field_device"
 				(path "/99623870-118f-49fe-bbf0-fb0b890db442/d15b20d6-817c-48cf-abc4-788b93984e6d"
-					(reference "#PWR041")
+					(reference "#PWR042")
 					(unit 1)
 				)
@@
 		(dnp no)
 		(fields_autoplaced yes)
-		(property "Reference" "C19"
+		(property "Reference" "C16"
 			(at 50.8 38.0999 0)
 			(show_name no)
@@
 			(project "field_device"
 				(path "/99623870-118f-49fe-bbf0-fb0b890db442/d15b20d6-817c-48cf-abc4-788b93984e6d"
-					(reference "C19")
+					(reference "C16")
 					(unit 1)
 				)
@@
 		(dnp no)
 		(fields_autoplaced yes)
-		(property "Reference" "#PWR035"
+		(property "Reference" "#PWR039"
 			(at 74.93 64.77 0)
 			(hide yes)
@@
 			(project "field_device"
 				(path "/99623870-118f-49fe-bbf0-fb0b890db442/d15b20d6-817c-48cf-abc4-788b93984e6d"
-					(reference "#PWR035")
+					(reference "#PWR039")
 					(unit 1)
 				)
@@
 		(in_pos_files yes)
 		(dnp no)
-		(property "Reference" "C23"
+		(property "Reference" "C21"
 			(at 172.72 42.672 90)
 			(show_name no)
@@
 			(project "field_device"
 				(path "/99623870-118f-49fe-bbf0-fb0b890db442/d15b20d6-817c-48cf-abc4-788b93984e6d"
-					(reference "C23")
+					(reference "C21")
 					(unit 1)
 				)
@@
 		(dnp no)
 		(fields_autoplaced yes)
-		(property "Reference" "C25"
+		(property "Reference" "C23"
 			(at 208.28 40.6399 0)
 			(show_name no)
@@
 			(project "field_device"
 				(path "/99623870-118f-49fe-bbf0-fb0b890db442/d15b20d6-817c-48cf-abc4-788b93984e6d"
-					(reference "C25")
+					(reference "C23")
 					(unit 1)
 				)
@@
 		(dnp no)
 		(fields_autoplaced yes)
-		(property "Reference" "#PWR048"
+		(property "Reference" "#PWR049"
 			(at 186.69 52.07 0)
 			(hide yes)
@@
 			(project "field_device"
 				(path "/99623870-118f-49fe-bbf0-fb0b890db442/d15b20d6-817c-48cf-abc4-788b93984e6d"
-					(reference "#PWR048")
+					(reference "#PWR049")
 					(unit 1)
 				)
@@
 		(dnp no)
 		(fields_autoplaced yes)
-		(property "Reference" "#PWR047"
+		(property "Reference" "#PWR048"
 			(at 143.51 31.75 0)
 			(hide yes)
@@
 			(project "field_device"
 				(path "/99623870-118f-49fe-bbf0-fb0b890db442/d15b20d6-817c-48cf-abc4-788b93984e6d"
-					(reference "#PWR047")
+					(reference "#PWR048")
 					(unit 1)
 				)
@@
 		(dnp no)
 		(fields_autoplaced yes)
-		(property "Reference" "#PWR046"
+		(property "Reference" "#PWR047"
 			(at 135.89 45.72 0)
 			(hide yes)
@@
 			(project "field_device"
 				(path "/99623870-118f-49fe-bbf0-fb0b890db442/d15b20d6-817c-48cf-abc4-788b93984e6d"
-					(reference "#PWR046")
+					(reference "#PWR047")
 					(unit 1)
 				)
@@
 		(dnp no)
 		(fields_autoplaced yes)
-		(property "Reference" "#PWR036"
+		(property "Reference" "#PWR037"
 			(at 22.86 39.37 0)
 			(hide yes)
@@
 			(project "field_device"
 				(path "/99623870-118f-49fe-bbf0-fb0b890db442/d15b20d6-817c-48cf-abc4-788b93984e6d"
-					(reference "#PWR036")
+					(reference "#PWR037")
 					(unit 1)
 				)
@@
 		(dnp no)
 		(fields_autoplaced yes)
-		(property "Reference" "C22"
+		(property "Reference" "C20"
 			(at 158.75 20.3199 0)
 			(show_name no)
@@
 			(project "field_device"
 				(path "/99623870-118f-49fe-bbf0-fb0b890db442/d15b20d6-817c-48cf-abc4-788b93984e6d"
-					(reference "C22")
+					(reference "C20")
 					(unit 1)
 				)
@@
 		(dnp no)
 		(fields_autoplaced yes)
-		(property "Reference" "#PWR039"
+		(property "Reference" "#PWR040"
 			(at 87.63 38.1 0)
 			(hide yes)
@@
 			(project "field_device"
 				(path "/99623870-118f-49fe-bbf0-fb0b890db442/d15b20d6-817c-48cf-abc4-788b93984e6d"
-					(reference "#PWR039")
+					(reference "#PWR040")
 					(unit 1)
 				)
@@
 		(dnp no)
 		(fields_autoplaced yes)
-		(property "Reference" "#PWR043"
+		(property "Reference" "#PWR044"
 			(at 135.89 33.02 0)
 			(hide yes)
@@
 			(project "field_device"
 				(path "/99623870-118f-49fe-bbf0-fb0b890db442/d15b20d6-817c-48cf-abc4-788b93984e6d"
-					(reference "#PWR043")
+					(reference "#PWR044")
 					(unit 1)
 				)
@@
 		(dnp no)
 		(fields_autoplaced yes)
-		(property "Reference" "C21"
+		(property "Reference" "C19"
 			(at 147.32 20.3199 0)
 			(show_name no)
@@
 			(project "field_device"
 				(path "/99623870-118f-49fe-bbf0-fb0b890db442/d15b20d6-817c-48cf-abc4-788b93984e6d"
-					(reference "C21")
+					(reference "C19")
 					(unit 1)
 				)
@@
 		(dnp no)
 		(fields_autoplaced yes)
-		(property "Reference" "C24"
+		(property "Reference" "C22"
 			(at 190.5 40.6399 0)
 			(show_name no)
@@
 			(project "field_device"
 				(path "/99623870-118f-49fe-bbf0-fb0b890db442/d15b20d6-817c-48cf-abc4-788b93984e6d"
-					(reference "C24")
+					(reference "C22")
 					(unit 1)
 				)
@@
 		(dnp no)
 		(fields_autoplaced yes)
-		(property "Reference" "C17"
+		(property "Reference" "C14"
 			(at 26.67 38.0999 0)
 			(show_name no)
@@
 			(project "field_device"
 				(path "/99623870-118f-49fe-bbf0-fb0b890db442/d15b20d6-817c-48cf-abc4-788b93984e6d"
-					(reference "C17")
+					(reference "C14")
 					(unit 1)
 				)
@@
 		(dnp no)
 		(fields_autoplaced yes)
-		(property "Reference" "#PWR044"
+		(property "Reference" "#PWR045"
 			(at 135.89 40.64 0)
 			(hide yes)
@@
 			(project "field_device"
 				(path "/99623870-118f-49fe-bbf0-fb0b890db442/d15b20d6-817c-48cf-abc4-788b93984e6d"
-					(reference "#PWR044")
+					(reference "#PWR045")
 					(unit 1)
 				)
@@
 		(dnp no)
 		(fields_autoplaced yes)
-		(property "Reference" "#PWR040"
+		(property "Reference" "#PWR041"
 			(at 87.63 45.72 0)
 			(hide yes)
@@
 			(project "field_device"
 				(path "/99623870-118f-49fe-bbf0-fb0b890db442/d15b20d6-817c-48cf-abc4-788b93984e6d"
-					(reference "#PWR040")
+					(reference "#PWR041")
 					(unit 1)
 				)
@@
 		(dnp no)
 		(fields_autoplaced yes)
-		(property "Reference" "C20"
+		(property "Reference" "C17"
 			(at 63.5 38.0999 0)
 			(show_name no)
@@
 			(project "field_device"
 				(path "/99623870-118f-49fe-bbf0-fb0b890db442/d15b20d6-817c-48cf-abc4-788b93984e6d"
-					(reference "C20")
+					(reference "C17")
 					(unit 1)
 				)
@@
 		(dnp no)
 		(fields_autoplaced yes)
-		(property "Reference" "C16"
+		(property "Reference" "C18"
 			(at 78.74 53.3399 0)
 			(show_name no)
@@
 			(project "field_device"
 				(path "/99623870-118f-49fe-bbf0-fb0b890db442/d15b20d6-817c-48cf-abc4-788b93984e6d"
-					(reference "C16")
+					(reference "C18")
 					(unit 1)
 				)
@@
 		(dnp no)
 		(fields_autoplaced yes)
-		(property "Reference" "C18"
+		(property "Reference" "C15"
 			(at 38.1 38.0999 0)
 			(show_name no)
@@
 			(project "field_device"
 				(path "/99623870-118f-49fe-bbf0-fb0b890db442/d15b20d6-817c-48cf-abc4-788b93984e6d"
-					(reference "C18")
+					(reference "C15")
 					(unit 1)
 				)
@@
 		(dnp no)
 		(fields_autoplaced yes)
-		(property "Reference" "#PWR037"
+		(property "Reference" "#PWR038"
 			(at 22.86 49.53 0)
 			(hide yes)
@@
 			(project "field_device"
 				(path "/99623870-118f-49fe-bbf0-fb0b890db442/d15b20d6-817c-48cf-abc4-788b93984e6d"
-					(reference "#PWR037")
+					(reference "#PWR038")
 					(unit 1)
 				)
@@
 		(dnp no)
 		(fields_autoplaced yes)
-		(property "Reference" "#PWR045"
+		(property "Reference" "#PWR046"
 			(at 135.89 43.18 0)
 			(hide yes)
@@
 			(project "field_device"
 				(path "/99623870-118f-49fe-bbf0-fb0b890db442/d15b20d6-817c-48cf-abc4-788b93984e6d"
-					(reference "#PWR045")
-					(unit 1)
-				)
+					(reference "#PWR046")
+					(unit 1)
+				)

Commit message: assigned better footprints
Parts:
- C14: footprint Capacitor_SMD:C_0603_1608Metric -> Capacitor_SMD:C_0805_2012Metric_Pad1.18x1.45mm_HandSolder
- C15, C16, C17, C18, C19: footprint Capacitor_SMD:C_0603_1608Metric -> Capacitor_SMD:C_0603_1608Metric_Pad1.08x0.95mm_HandSolder
- C20, C22, C23: footprint Capacitor_SMD:C_0603_1608Metric -> Capacitor_SMD:C_0402_1005Metric_Pad0.74x0.62mm_HandSolder
Other:
- moved on the sheet: Y1
Changed lines of the file:
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@@
 	)
 	(rectangle
-		(start -10.16 27.94)
-		(end 7.62 52.07)
+		(start 16.51 55.88)
+		(end 34.29 80.01)
 		(stroke
 			(width 0)
@@
 	(text "Crystal"
 		(exclude_from_sim no)
-		(at -1.016 53.594 0)
+		(at 25.654 81.534 0)
 		(effects
 			(font
@@
 	)
 	(label "XTA"
-		(at 2.54 39.37 0)
+		(at 29.21 67.31 0)
 		(effects
 			(font
@@
 	)
 	(label "XTB"
-		(at -5.08 39.37 180)
+		(at 21.59 67.31 180)
 		(effects
 			(font
@@
 	(symbol
 		(lib_id "power:GND")
-		(at -1.27 44.45 0)
+		(at 25.4 72.39 0)
 		(unit 1)
 		(body_style 1)
@@
 		(fields_autoplaced yes)
 		(property "Reference" "#PWR036"
-			(at -1.27 50.8 0)
+			(at 25.4 78.74 0)
 			(hide yes)
 			(show_name no)
@@
 		)
 		(property "Value" "GND"
-			(at -1.27 49.53 0)
+			(at 25.4 77.47 0)
 			(show_name no)
 			(do_not_autoplace no)
@@
 		)
 		(property "Footprint" ""
-			(at -1.27 44.45 0)
+			(at 25.4 72.39 0)
 			(hide yes)
 			(show_name no)
@@
 		)
 		(property "Datasheet" ""
-			(at -1.27 44.45 0)
+			(at 25.4 72.39 0)
 			(hide yes)
 			(show_name no)
@@
 		)
 		(property "Description" "Power symbol creates a global label with name \"GND\" , ground"
-			(at -1.27 44.45 0)
+			(at 25.4 72.39 0)
 			(hide yes)
 			(show_name no)
@@
 	(symbol
 		(lib_id "Device:Crystal_GND24")
-		(at -1.27 39.37 0)
+		(at 25.4 67.31 0)
 		(unit 1)
 		(body_style 1)
@@
 		(fields_autoplaced yes)
 		(property "Reference" "Y1"
-			(at -1.27 30.48 0)
+			(at 25.4 58.42 0)
 			(show_name no)
 			(do_not_autoplace no)
@@
 		)
 		(property "Value" "Crystal_GND24"
-			(at -1.27 33.02 0)
+			(at 25.4 60.96 0)
 			(show_name no)
 			(do_not_autoplace no)
@@
 		)
 		(property "Footprint" "Crystal:Crystal_SMD_3225-4Pin_3.2x2.5mm"
-			(at -1.27 39.37 0)
+			(at 25.4 67.31 0)
 			(hide yes)
 			(show_name no)
@@
 		)
 		(property "Datasheet" ""
-			(at -1.27 39.37 0)
+			(at 25.4 67.31 0)
 			(hide yes)
 			(show_name no)
@@
 		)
 		(property "Description" "Four pin crystal, GND on pins 2 and 4"
-			(at -1.27 39.37 0)
+			(at 25.4 67.31 0)
 			(hide yes)
 			(show_name no)
@@
 		)
 		(property private "KLC_S3.3" "The rectangle is not a symbol body but a graphical element"
-			(at -1.27 52.07 0)
+			(at 25.4 80.01 0)
 			(hide yes)
 			(show_name yes)
@@
 		)
 		(property private "KLC_S4.1" "Some pins are on 50mil grid to make the symbol small"
-			(at -1.27 54.61 0)
+			(at 25.4 82.55 0)
 			(hide yes)
 			(show_name yes)
@@
 			)
 		)
-		(property "Footprint" "Capacitor_SMD:C_0603_1608Metric"
+		(property "Footprint" "Capacitor_SMD:C_0603_1608Metric_Pad1.08x0.95mm_HandSolder"
 			(at 47.9552 43.18 0)
 			(hide yes)
@@
 			)
 		)
-		(property "Footprint" "Capacitor_SMD:C_0603_1608Metric"
+		(property "Footprint" "Capacitor_SMD:C_0402_1005Metric_Pad0.74x0.62mm_HandSolder"
 			(at 205.4352 45.72 0)
 			(hide yes)
@@
 			)
 		)
-		(property "Footprint" "Capacitor_SMD:C_0603_1608Metric"
+		(property "Footprint" "Capacitor_SMD:C_0402_1005Metric_Pad0.74x0.62mm_HandSolder"
 			(at 155.9052 25.4 0)
 			(hide yes)
@@
 			)
 		)
-		(property "Footprint" "Capacitor_SMD:C_0603_1608Metric"
+		(property "Footprint" "Capacitor_SMD:C_0603_1608Metric_Pad1.08x0.95mm_HandSolder"
 			(at 144.4752 25.4 0)
 			(hide yes)
@@
 			)
 		)
-		(property "Footprint" "Capacitor_SMD:C_0603_1608Metric"
+		(property "Footprint" "Capacitor_SMD:C_0402_1005Metric_Pad0.74x0.62mm_HandSolder"
 			(at 187.6552 45.72 0)
 			(hide yes)
@@
 			)
 		)
-		(property "Footprint" "Capacitor_SMD:C_0603_1608Metric"
+		(property "Footprint" "Capacitor_SMD:C_0805_2012Metric_Pad1.18x1.45mm_HandSolder"
 			(at 23.8252 43.18 0)
 			(hide yes)
@@
 			)
 		)
-		(property "Footprint" "Capacitor_SMD:C_0603_1608Metric"
+		(property "Footprint" "Capacitor_SMD:C_0603_1608Metric_Pad1.08x0.95mm_HandSolder"
 			(at 60.6552 43.18 0)
 			(hide yes)
@@
 			)
 		)
-		(property "Footprint" "Capacitor_SMD:C_0603_1608Metric"
+		(property "Footprint" "Capacitor_SMD:C_0603_1608Metric_Pad1.08x0.95mm_HandSolder"
 			(at 75.8952 58.42 0)
 			(hide yes)
@@
 			)
 		)
-		(property "Footprint" "Capacitor_SMD:C_0603_1608Metric"
+		(property "Footprint" "Capacitor_SMD:C_0603_1608Metric_Pad1.08x0.95mm_HandSolder"
 			(at 35.2552 43.18 0)
 			(hide yes)

Commit message: changed regulator
Parts:
- C13: renamed from C14; footprint Capacitor_SMD:C_0805_2012Metric_Pad1.18x1.45mm_HandSolder -> Capacitor_SMD:C_0603_1608Metric_Pad1.08x0.95mm_HandSolder
- C14: renamed from C15; footprint Capacitor_SMD:C_0603_1608Metric_Pad1.08x0.95mm_HandSolder -> Capacitor_SMD:C_0402_1005Metric_Pad0.74x0.62mm_HandSolder
- C15: renamed from C16; footprint Capacitor_SMD:C_0603_1608Metric_Pad1.08x0.95mm_HandSolder -> Capacitor_SMD:C_0402_1005Metric_Pad0.74x0.62mm_HandSolder
- C16: renamed from C17; footprint Capacitor_SMD:C_0603_1608Metric_Pad1.08x0.95mm_HandSolder -> Capacitor_SMD:C_0402_1005Metric_Pad0.74x0.62mm_HandSolder
- C18: renamed from C19; footprint Capacitor_SMD:C_0603_1608Metric_Pad1.08x0.95mm_HandSolder -> Capacitor_SMD:C_0402_1005Metric_Pad0.74x0.62mm_HandSolder
- C20: renamed from C21; footprint Capacitor_SMD:C_0603_1608Metric -> Capacitor_SMD:C_0402_1005Metric_Pad0.74x0.62mm_HandSolder
- L2, L3: footprint Inductor_SMD:L_0603_1608Metric -> Inductor_SMD:L_0402_1005Metric_Pad0.77x0.64mm_HandSolder
- renumbered C18 to C17, C20 to C19, C22 to C21, C23 to C22
Changed lines of the file:
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@@
 		(dnp no)
 		(fields_autoplaced yes)
-		(property "Reference" "#PWR036"
+		(property "Reference" "#PWR038"
 			(at 25.4 78.74 0)
 			(hide yes)
@@
 			(project "field_device"
 				(path "/99623870-118f-49fe-bbf0-fb0b890db442/d15b20d6-817c-48cf-abc4-788b93984e6d"
-					(reference "#PWR036")
+					(reference "#PWR038")
 					(unit 1)
 				)
@@
 		(dnp no)
 		(fields_autoplaced yes)
-		(property "Reference" "C16"
+		(property "Reference" "C15"
 			(at 50.8 38.0999 0)
 			(show_name no)
@@
 			)
 		)
-		(property "Footprint" "Capacitor_SMD:C_0603_1608Metric_Pad1.08x0.95mm_HandSolder"
+		(property "Footprint" "Capacitor_SMD:C_0402_1005Metric_Pad0.74x0.62mm_HandSolder"
 			(at 47.9552 43.18 0)
 			(hide yes)
@@
 			(project "field_device"
 				(path "/99623870-118f-49fe-bbf0-fb0b890db442/d15b20d6-817c-48cf-abc4-788b93984e6d"
-					(reference "C16")
+					(reference "C15")
 					(unit 1)
 				)
@@
 		(in_pos_files yes)
 		(dnp no)
-		(property "Reference" "C21"
+		(property "Reference" "C20"
 			(at 172.72 42.672 90)
 			(show_name no)
@@
 			)
 		)
-		(property "Footprint" "Capacitor_SMD:C_0603_1608Metric"
+		(property "Footprint" "Capacitor_SMD:C_0402_1005Metric_Pad0.74x0.62mm_HandSolder"
 			(at 168.91 39.0652 0)
 			(hide yes)
@@
 			(project "field_device"
 				(path "/99623870-118f-49fe-bbf0-fb0b890db442/d15b20d6-817c-48cf-abc4-788b93984e6d"
-					(reference "C21")
+					(reference "C20")
 					(unit 1)
 				)
@@
 		(dnp no)
 		(fields_autoplaced yes)
-		(property "Reference" "C23"
+		(property "Reference" "C22"
 			(at 208.28 40.6399 0)
 			(show_name no)
@@
 			(project "field_device"
 				(path "/99623870-118f-49fe-bbf0-fb0b890db442/d15b20d6-817c-48cf-abc4-788b93984e6d"
-					(reference "C23")
+					(reference "C22")
 					(unit 1)
 				)
@@
 		(dnp no)
 		(fields_autoplaced yes)
-		(property "Reference" "#PWR037"
+		(property "Reference" "#PWR036"
 			(at 22.86 39.37 0)
 			(hide yes)
@@
 			(project "field_device"
 				(path "/99623870-118f-49fe-bbf0-fb0b890db442/d15b20d6-817c-48cf-abc4-788b93984e6d"
-					(reference "#PWR037")
+					(reference "#PWR036")
 					(unit 1)
 				)
@@
 			)
 		)
-		(property "Footprint" "Inductor_SMD:L_0603_1608Metric"
+		(property "Footprint" "Inductor_SMD:L_0402_1005Metric_Pad0.77x0.64mm_HandSolder"
 			(at 166.37 21.59 0)
 			(hide yes)
@@
 		(dnp no)
 		(fields_autoplaced yes)
-		(property "Reference" "C20"
+		(property "Reference" "C19"
 			(at 158.75 20.3199 0)
 			(show_name no)
@@
 			(project "field_device"
 				(path "/99623870-118f-49fe-bbf0-fb0b890db442/d15b20d6-817c-48cf-abc4-788b93984e6d"
-					(reference "C20")
+					(reference "C19")
 					(unit 1)
 				)
@@
 		(dnp no)
 		(fields_autoplaced yes)
-		(property "Reference" "C19"
+		(property "Reference" "C18"
 			(at 147.32 20.3199 0)
 			(show_name no)
@@
 			)
 		)
-		(property "Footprint" "Capacitor_SMD:C_0603_1608Metric_Pad1.08x0.95mm_HandSolder"
+		(property "Footprint" "Capacitor_SMD:C_0402_1005Metric_Pad0.74x0.62mm_HandSolder"
 			(at 144.4752 25.4 0)
 			(hide yes)
@@
 			(project "field_device"
 				(path "/99623870-118f-49fe-bbf0-fb0b890db442/d15b20d6-817c-48cf-abc4-788b93984e6d"
-					(reference "C19")
+					(reference "C18")
 					(unit 1)
 				)
@@
 		(dnp no)
 		(fields_autoplaced yes)
-		(property "Reference" "C22"
+		(property "Reference" "C21"
 			(at 190.5 40.6399 0)
 			(show_name no)
@@
 			(project "field_device"
 				(path "/99623870-118f-49fe-bbf0-fb0b890db442/d15b20d6-817c-48cf-abc4-788b93984e6d"
-					(reference "C22")
+					(reference "C21")
 					(unit 1)
 				)
@@
 		(dnp no)
 		(fields_autoplaced yes)
-		(property "Reference" "C14"
+		(property "Reference" "C13"
 			(at 26.67 38.0999 0)
 			(show_name no)
@@
 			)
 		)
-		(property "Footprint" "Capacitor_SMD:C_0805_2012Metric_Pad1.18x1.45mm_HandSolder"
+		(property "Footprint" "Capacitor_SMD:C_0603_1608Metric_Pad1.08x0.95mm_HandSolder"
 			(at 23.8252 43.18 0)
 			(hide yes)
@@
 			(project "field_device"
 				(path "/99623870-118f-49fe-bbf0-fb0b890db442/d15b20d6-817c-48cf-abc4-788b93984e6d"
-					(reference "C14")
+					(reference "C13")
 					(unit 1)
 				)
@@
 			)
 		)
-		(property "Footprint" "Inductor_SMD:L_0603_1608Metric"
+		(property "Footprint" "Inductor_SMD:L_0402_1005Metric_Pad0.77x0.64mm_HandSolder"
 			(at 195.58 38.1 0)
 			(hide yes)
@@
 		(dnp no)
 		(fields_autoplaced yes)
-		(property "Reference" "C17"
+		(property "Reference" "C16"
 			(at 63.5 38.0999 0)
 			(show_name no)
@@
 			)
 		)
-		(property "Footprint" "Capacitor_SMD:C_0603_1608Metric_Pad1.08x0.95mm_HandSolder"
+		(property "Footprint" "Capacitor_SMD:C_0402_1005Metric_Pad0.74x0.62mm_HandSolder"
 			(at 60.6552 43.18 0)
 			(hide yes)
@@
 			(project "field_device"
 				(path "/99623870-118f-49fe-bbf0-fb0b890db442/d15b20d6-817c-48cf-abc4-788b93984e6d"
-					(reference "C17")
+					(reference "C16")
 					(unit 1)
 				)
@@
 		(dnp no)
 		(fields_autoplaced yes)
-		(property "Reference" "C18"
+		(property "Reference" "C17"
 			(at 78.74 53.3399 0)
 			(show_name no)
@@
 			(project "field_device"
 				(path "/99623870-118f-49fe-bbf0-fb0b890db442/d15b20d6-817c-48cf-abc4-788b93984e6d"
-					(reference "C18")
+					(reference "C17")
 					(unit 1)
 				)
@@
 		(dnp no)
 		(fields_autoplaced yes)
-		(property "Reference" "C15"
+		(property "Reference" "C14"
 			(at 38.1 38.0999 0)
 			(show_name no)
@@
 			)
 		)
-		(property "Footprint" "Capacitor_SMD:C_0603_1608Metric_Pad1.08x0.95mm_HandSolder"
+		(property "Footprint" "Capacitor_SMD:C_0402_1005Metric_Pad0.74x0.62mm_HandSolder"
 			(at 35.2552 43.18 0)
 			(hide yes)
@@
 			(project "field_device"
 				(path "/99623870-118f-49fe-bbf0-fb0b890db442/d15b20d6-817c-48cf-abc4-788b93984e6d"
-					(reference "C15")
+					(reference "C14")
 					(unit 1)
 				)
@@
 		(dnp no)
 		(fields_autoplaced yes)
-		(property "Reference" "#PWR038"
+		(property "Reference" "#PWR037"
 			(at 22.86 49.53 0)
 			(hide yes)
@@
 			(project "field_device"
 				(path "/99623870-118f-49fe-bbf0-fb0b890db442/d15b20d6-817c-48cf-abc4-788b93984e6d"
-					(reference "#PWR038")
-					(unit 1)
-				)
+					(reference "#PWR037")
+					(unit 1)
+				)
