File: boards/field_device/lora_module.kicad_sch (KiCad schematic)
At the start: 15 parts, among them U6 SX1262IMLTRT, Y1 X322532MMB4SI

Commit message: rev 5?
Parts:
- removed AE1: Antenna, custom:TI DN023 868-955MHz Antenna, symbol Device:Antenna
- removed C16: 100nF, Capacitor_SMD:C_0402_1005Metric_Pad0.74x0.62mm_HandSolder, symbol Device:C
- added AE1: monopole, custom:TI DN023 868-955MHz Antenna, symbol Device:Antenna_Shield
- added C12: 10u, Capacitor_SMD:C_0603_1608Metric_Pad1.08x0.95mm_HandSolder, symbol Device:C
- C11: renamed from C17; value 470nF -> 10u
- C13: value 10uF -> 10u
- C14: renamed from C15; value 100nF -> 100n
- C15: renamed from C14; value 100nF -> 100n
- C16: renamed from C18; value 47nF -> 47n; footprint Capacitor_SMD:C_0402_1005Metric_Pad0.74x0.62mm_HandSolder -> Capacitor_SMD:C_0402_1005Metric
- C17: renamed from C19; value 100pF -> 100p; footprint Capacitor_SMD:C_0402_1005Metric_Pad0.74x0.62mm_HandSolder -> Capacitor_SMD:C_0402_1005Metric
- C18: renamed from C20; value 100pF -> 100p
- L2: value 47nH -> 47n
- renumbered C21 to C19, C22 to C20, R17 to R15
Connections:
- net +3.3V: now also C12.1
- net GND: now also AE1.2 (Shield), C12.2; no longer C20.1, R15.2
- net RFO: now reaches C18.1, C19.1, R15.1
- net RFO: now also C18.2, C20.1, L2.2, R15.2, U6.23 (RFO), AE1.1 (A)
- net VR_PA: now reaches C16.1, C17.1, L2.1, U6.24 (VR_PA)
- net VREG: now reaches C11.1, U6.7 (VREG)
Other:
- title: (none) -> Field Device RF communications
- moved on the sheet: C11, C13, C14, C15, C16, C17, Y1

Commit message: change components to fit manufacturing capability
Parts:
- C11, C12, C13: value 10u -> 10uF
- C14, C15: value 100n -> 100nF
- C16: value 47n -> 47nF C0G; footprint Capacitor_SMD:C_0402_1005Metric -> Resistor_SMD:R_1206_3216Metric
- C17, C18: value 100p -> 100p C0G
- L2: value 47n -> 47nH VHF100505HQ47NJT
Changed lines of the file:
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@@
 			)
 		)
-		(property "Value" "100n"
+		(property "Value" "100nF"
 			(at 73.66 63.4999 0)
 			(show_name no)
@@
 			)
 		)
-		(property "Value" "100p"
+		(property "Value" "100p C0G"
 			(at 172.72 45.212 90)
 			(show_name no)
@@
 			)
 		)
-		(property "Value" "47n"
+		(property "Value" "47nH VHF100505HQ47NJT"
 			(at 167.64 22.8599 0)
 			(show_name no)
@@
 		(in_pos_files yes)
 		(dnp no)
-		(fields_autoplaced yes)
 		(property "Reference" "C17"
 			(at 147.32 20.3199 0)
@@
 			)
 		)
-		(property "Value" "100p"
-			(at 147.32 22.8599 0)
+		(property "Value" "100p C0G"
+			(at 145.796 26.924 0)
 			(show_name no)
 			(do_not_autoplace no)
@@
 			)
 		)
-		(property "Value" "10u"
+		(property "Value" "10uF"
 			(at 62.23 63.4999 0)
 			(show_name no)
@@
 		(in_pos_files yes)
 		(dnp no)
-		(fields_autoplaced yes)
 		(property "Reference" "C16"
 			(at 160.02 20.3199 0)
@@
 			)
 		)
-		(property "Value" "47n"
-			(at 160.02 22.8599 0)
+		(property "Value" "47nF C0G"
+			(at 156.21 26.924 0)
 			(show_name no)
 			(do_not_autoplace no)
@@
 			)
 		)
-		(property "Footprint" "Capacitor_SMD:C_0402_1005Metric"
+		(property "Footprint" "Resistor_SMD:R_1206_3216Metric"
 			(at 157.1752 25.4 0)
 			(hide yes)
@@
 			)
 		)
-		(property "Value" "10u"
+		(property "Value" "10uF"
 			(at 64.77 40.6399 0)
 			(show_name no)
@@
 			)
 		)
-		(property "Value" "10u"
+		(property "Value" "10uF"
 			(at 45.72 55.8799 0)
 			(show_name no)
@@
 			)
 		)
-		(property "Value" "100n"
+		(property "Value" "100nF"
 			(at 76.2 40.6399 0)
 			(show_name no)

Commit message: idk atp
Parts:
- C11, C12, C13: value 10uF -> CL10A106KP8NNNC 10uF
- C14, C15: value 100nF -> CL05B104KO5NNNC 100nF
- C16: value 47nF C0G -> 47nF
- C17, C18: value 100p C0G -> 0402CG101J500NT 100pF
- L2: value 47nH VHF100505HQ47NJT -> 47nH; footprint Inductor_SMD:L_0402_1005Metric_Pad0.77x0.64mm_HandSolder -> Inductor_SMD:L_0805_2012Metric_Pad1.05x1.20mm_HandSolder
Changed lines of the file:
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@@
 			)
 		)
-		(property "Value" "100nF"
+		(property "Value" "CL05B104KO5NNNC 100nF"
 			(at 73.66 63.4999 0)
 			(show_name no)
@@
 			)
 		)
-		(property "Value" "100p C0G"
+		(property "Value" "0402CG101J500NT 100pF"
 			(at 172.72 45.212 90)
 			(show_name no)
@@
 			)
 		)
-		(property "Value" "47nH VHF100505HQ47NJT"
+		(property "Value" "47nH"
 			(at 167.64 22.8599 0)
 			(show_name no)
@@
 			)
 		)
-		(property "Footprint" "Inductor_SMD:L_0402_1005Metric_Pad0.77x0.64mm_HandSolder"
+		(property "Footprint" "Inductor_SMD:L_0805_2012Metric_Pad1.05x1.20mm_HandSolder"
 			(at 166.37 21.59 0)
 			(hide yes)
@@
 			)
 		)
-		(property "Value" "100p C0G"
-			(at 145.796 26.924 0)
+		(property "Value" "0402CG101J500NT 100pF"
+			(at 145.034 28.956 0)
 			(show_name no)
 			(do_not_autoplace no)
@@
 			)
 		)
-		(property "Value" "10uF"
+		(property "Value" "CL10A106KP8NNNC 10uF"
 			(at 62.23 63.4999 0)
 			(show_name no)
@@
 			)
 		)
-		(property "Value" "47nF C0G"
+		(property "Value" "47nF"
 			(at 156.21 26.924 0)
 			(show_name no)
@@
 			)
 		)
-		(property "Value" "10uF"
+		(property "Value" "CL10A106KP8NNNC 10uF"
 			(at 64.77 40.6399 0)
 			(show_name no)
@@
 			)
 		)
-		(property "Value" "10uF"
+		(property "Value" "CL10A106KP8NNNC 10uF"
 			(at 45.72 55.8799 0)
 			(show_name no)
@@
 			)
 		)
-		(property "Value" "100nF"
+		(property "Value" "CL05B104KO5NNNC 100nF"
 			(at 76.2 40.6399 0)
 			(show_name no)

Commit message: peer review
Parts:
- C16: footprint Resistor_SMD:R_1206_3216Metric -> Capacitor_SMD:C_0603_1608Metric
- C17: value 0402CG101J500NT 100pF -> CL05B104KO5NNNC 100nF
Changed lines of the file:
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@@
 			)
 		)
-		(property "Value" "0402CG101J500NT 100pF"
+		(property "Value" "CL05B104KO5NNNC 100nF"
 			(at 145.034 28.956 0)
 			(show_name no)
@@
 			)
 		)
-		(property "Footprint" "Resistor_SMD:R_1206_3216Metric"
+		(property "Footprint" "Capacitor_SMD:C_0603_1608Metric"
 			(at 157.1752 25.4 0)
 			(hide yes)
