File: boards/field_device/power_source.kicad_sch (KiCad schematic)
At the start: 9 parts, among them U4 CN3163

Commit message: route more stuff
Parts:
- R15: footprint Resistor_SMD:R_0603_1608Metric -> Capacitor_SMD:C_0603_1608Metric_Pad1.08x0.95mm_HandSolder
Changed lines of the file:
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@@
 			)
 		)
-		(property "Footprint" "Resistor_SMD:R_0603_1608Metric"
+		(property "Footprint" "Capacitor_SMD:C_0603_1608Metric_Pad1.08x0.95mm_HandSolder"
 			(at 72.39 79.248 90)
 			(hide yes)
