File: boards/field_device/power_source.kicad_sch (KiCad schematic)
At the start: 9 parts, among them U4 CN3163

Commit message: rev 5?
Parts:
- renumbered R14 to R11, R15 to R12
Connections:
- net ISET: now reaches R11.1, U4.2 (ISET)
Other:
- title: (none) -> Field Device Power Supply
Changed lines of the file:
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@@
 	(generator_version "10.0")
 	(paper "A4")
+	(title_block
+		(title "Field Device Power Supply")
+		(date "2026-10-09")
+		(rev "5")
+	)
 	(junction
 		(at 106.68 55.88)
@@
 	(wire
 		(pts
-			(xy 62.23 77.47) (xy 68.58 77.47)
+			(xy 72.39 40.64) (xy 81.28 40.64)
 		)
 		(stroke
@@
 	(wire
 		(pts
-			(xy 104.14 45.72) (xy 118.11 45.72)
+			(xy 62.23 77.47) (xy 68.58 77.47)
 		)
 		(stroke
@@
 	(wire
 		(pts
-			(xy 81.28 40.64) (xy 72.39 40.64)
+			(xy 104.14 45.72) (xy 118.11 45.72)
 		)
 		(stroke
@@
 			)
 			(justify left bottom)
+		)
+	)
+	(label "ISET"
+		(at 77.47 40.64 180)
+		(effects
+			(font
+				(size 1.27 1.27)
+			)
+			(justify right bottom)
 		)
 	)
@@
 		(dnp no)
 		(fields_autoplaced yes)
-		(property "Reference" "#PWR020"
+		(property "Reference" "#PWR018"
 			(at 48.26 59.69 0)
 			(hide yes)
@@
 			(project "field_device"
 				(path "/99623870-118f-49fe-bbf0-fb0b890db442/e9c11804-cc5e-4b00-a5de-7502c32ebb51"
-					(reference "#PWR020")
+					(reference "#PWR018")
 					(unit 1)
 				)
@@
 		(dnp no)
 		(fields_autoplaced yes)
-		(property "Reference" "#PWR022"
+		(property "Reference" "#PWR020"
 			(at 74.93 38.1 0)
 			(hide yes)
@@
 			(project "field_device"
 				(path "/99623870-118f-49fe-bbf0-fb0b890db442/e9c11804-cc5e-4b00-a5de-7502c32ebb51"
-					(reference "#PWR022")
+					(reference "#PWR020")
 					(unit 1)
 				)
@@
 		(dnp no)
 		(fields_autoplaced yes)
-		(property "Reference" "#PWR019"
+		(property "Reference" "#PWR017"
 			(at 30.48 59.69 0)
 			(hide yes)
@@
 			(project "field_device"
 				(path "/99623870-118f-49fe-bbf0-fb0b890db442/e9c11804-cc5e-4b00-a5de-7502c32ebb51"
-					(reference "#PWR019")
+					(reference "#PWR017")
 					(unit 1)
 				)
@@
 		(dnp no)
 		(fields_autoplaced yes)
-		(property "Reference" "#PWR021"
+		(property "Reference" "#PWR019"
 			(at 72.39 68.58 0)
 			(hide yes)
@@
 			(project "field_device"
 				(path "/99623870-118f-49fe-bbf0-fb0b890db442/e9c11804-cc5e-4b00-a5de-7502c32ebb51"
-					(reference "#PWR021")
+					(reference "#PWR019")
 					(unit 1)
 				)
@@
 		(dnp no)
 		(fields_autoplaced yes)
-		(property "Reference" "#PWR024"
+		(property "Reference" "#PWR022"
 			(at 92.71 24.13 0)
 			(hide yes)
@@
 			(project "field_device"
 				(path "/99623870-118f-49fe-bbf0-fb0b890db442/e9c11804-cc5e-4b00-a5de-7502c32ebb51"
-					(reference "#PWR024")
+					(reference "#PWR022")
 					(unit 1)
 				)
@@
 		(dnp no)
 		(fields_autoplaced yes)
-		(property "Reference" "R15"
+		(property "Reference" "R12"
 			(at 72.39 71.12 90)
 			(show_name no)
@@
 			(project "field_device"
 				(path "/99623870-118f-49fe-bbf0-fb0b890db442/e9c11804-cc5e-4b00-a5de-7502c32ebb51"
-					(reference "R15")
+					(reference "R12")
 					(unit 1)
 				)
@@
 		(dnp no)
 		(fields_autoplaced yes)
-		(property "Reference" "#PWR025"
+		(property "Reference" "#PWR023"
 			(at 106.68 62.23 0)
 			(hide yes)
@@
 			(project "field_device"
 				(path "/99623870-118f-49fe-bbf0-fb0b890db442/e9c11804-cc5e-4b00-a5de-7502c32ebb51"
-					(reference "#PWR025")
+					(reference "#PWR023")
 					(unit 1)
 				)
@@
 		(dnp no)
 		(fields_autoplaced yes)
-		(property "Reference" "#PWR023"
+		(property "Reference" "#PWR021"
 			(at 74.93 43.18 0)
 			(hide yes)
@@
 			(project "field_device"
 				(path "/99623870-118f-49fe-bbf0-fb0b890db442/e9c11804-cc5e-4b00-a5de-7502c32ebb51"
-					(reference "#PWR023")
+					(reference "#PWR021")
 					(unit 1)
 				)
@@
 		(dnp no)
 		(fields_autoplaced yes)
-		(property "Reference" "R14"
+		(property "Reference" "R11"
 			(at 74.93 57.1499 0)
 			(show_name no)
@@
 			(project "field_device"
 				(path "/99623870-118f-49fe-bbf0-fb0b890db442/e9c11804-cc5e-4b00-a5de-7502c32ebb51"
-					(reference "R14")
+					(reference "R11")
 					(unit 1)
 				)

Commit message: idk atp
Parts:
- C7, C8: value 10uF -> CL10A106KP8NNNC 10uF
Changed lines of the file:
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@@
 			)
 		)
-		(property "Value" "10uF"
+		(property "Value" "CL10A106KP8NNNC 10uF"
 			(at 110.49 52.0699 0)
 			(show_name no)
@@
 			)
 		)
-		(property "Value" "10uF"
+		(property "Value" "CL10A106KP8NNNC 10uF"
 			(at 52.07 50.7999 0)
 			(show_name no)
