File: boards/field_device/mcu.kicad_sch (KiCad schematic)
At the start: 19 parts, among them J1 Conn_01x05_Pin, J2 Conn_01x02_Pin, SW1 SW_SPST, U2 STM32C011F6Px

Commit message: changed regulator
Parts:
- removed C5: 100n, Capacitor_SMD:C_0603_1608Metric_Pad1.08x0.95mm_HandSolder, symbol Device:C
- added R5: 22R, Resistor_SMD:R_0402_1005Metric_Pad0.72x0.64mm_HandSolder, symbol Device:R
- C2, C4: footprint Capacitor_SMD:C_0603_1608Metric_Pad1.08x0.95mm_HandSolder -> Capacitor_SMD:C_0402_1005Metric_Pad0.74x0.62mm_HandSolder
- C3: footprint Capacitor_SMD:C_0805_2012Metric_Pad1.18x1.45mm_HandSolder -> Capacitor_SMD:C_0603_1608Metric_Pad1.08x0.95mm_HandSolder
- R12: renamed from R11; footprint Resistor_SMD:R_0603_1608Metric -> Resistor_SMD:R_0402_1005Metric_Pad0.72x0.64mm_HandSolder
- renumbered R9 to R10, R10 to R11, R5 to R6, R6 to R7, R7 to R8, R8 to R9
Connections:
- net RF_NSS: now also R5.1, R5.2
Other:
- moved on the sheet: C3, C4

Commit message: routed everything
Parts:
- R3: footprint Resistor_SMD:R_0402_1005Metric_Pad0.72x0.64mm_HandSolder -> Resistor_SMD:R_0603_1608Metric_Pad0.98x0.95mm_HandSolder
Connections:
- net +3.3V: now also J1.4 (Pin_4); no longer J1.2 (Pin_2)
- net GND: now also J1.3 (Pin_3); no longer J1.1 (Pin_1)
- net RF_MISO: no longer R7.1, U2.13 (PA6)
- net RF_MOSI: no longer R8.1, U2.14 (PA7)
- net RF_NSS: no longer R5.1, U2.11 (PA4)
- net RF_SCK: no longer R6.1, U2.12 (PA5)
- net SWDCLK: now also J1.2 (Pin_2); no longer J1.3 (Pin_3)
- net SWDIO: now also J1.1 (Pin_1); no longer J1.4 (Pin_4)
- new net MCU_MISO: R7.1, U2.13 (PA6)
- new net MCU_MOSI: R8.1, U2.14 (PA7)
- new net MCU_NSS: R5.1, U2.11 (PA4)
- new net MCU_SCK: R6.1, U2.12 (PA5)
Changed lines of the file:
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@@
+	(wire
+		(pts
+			(xy 96.52 69.85) (xy 46.99 69.85)
+		)
+		(stroke
+			(width 0)
+			(type default)
+		)
+	)
 	(wire
 		(pts
@@
 	(wire
 		(pts
-			(xy 96.52 77.47) (xy 46.99 77.47)
-		)
-		(stroke
-			(width 0)
-			(type default)
-		)
-	)
-	(wire
-		(pts
 			(xy 170.18 69.85) (xy 207.01 69.85)
 		)
@@
 	(wire
 		(pts
-			(xy 99.06 74.93) (xy 99.06 87.63)
+			(xy 73.66 111.76) (xy 87.63 111.76)
+		)
+		(stroke
+			(width 0)
+			(type default)
+		)
+	)
+	(wire
+		(pts
+			(xy 57.15 44.45) (xy 109.22 44.45)
+		)
+		(stroke
+			(width 0)
+			(type default)
+		)
+	)
+	(wire
+		(pts
+			(xy 170.18 67.31) (xy 207.01 67.31)
+		)
+		(stroke
+			(width 0)
+			(type default)
+		)
+	)
+	(wire
+		(pts
+			(xy 96.52 91.44) (xy 148.59 91.44)
+		)
+		(stroke
+			(width 0)
+			(type default)
+		)
+	)
+	(wire
+		(pts
+			(xy 97.79 27.94) (xy 127 27.94)
+		)
+		(stroke
+			(width 0)
+			(type default)
+		)
+	)
+	(wire
+		(pts
+			(xy 149.86 76.2) (xy 170.18 76.2)
+		)
+		(stroke
+			(width 0)
+			(type default)
+		)
+	)
+	(wire
+		(pts
+			(xy 170.18 54.61) (xy 191.77 54.61)
+		)
+		(stroke
+			(width 0)
+			(type default)
+		)
+	)
+	(wire
+		(pts
+			(xy 46.99 72.39) (xy 99.06 72.39)
+		)
+		(stroke
+			(width 0)
+			(type default)
+		)
+	)
+	(wire
+		(pts
+			(xy 104.14 57.15) (xy 109.22 57.15)
+		)
+		(stroke
+			(width 0)
+			(type default)
+		)
+	)
+	(wire
+		(pts
+			(xy 96.52 91.44) (xy 96.52 69.85)
+		)
+		(stroke
+			(width 0)
+			(type default)
+		)
+	)
+	(wire
+		(pts
+			(xy 99.06 72.39) (xy 99.06 87.63)
 		)
 		(stroke
@@
 		(pts
 			(xy 46.99 80.01) (xy 57.15 80.01)
-		)
-		(stroke
-			(width 0)
-			(type default)
-		)
-	)
-	(wire
-		(pts
-			(xy 73.66 111.76) (xy 87.63 111.76)
-		)
-		(stroke
-			(width 0)
-			(type default)
-		)
-	)
-	(wire
-		(pts
-			(xy 57.15 44.45) (xy 109.22 44.45)
-		)
-		(stroke
-			(width 0)
-			(type default)
-		)
-	)
-	(wire
-		(pts
-			(xy 170.18 67.31) (xy 207.01 67.31)
-		)
-		(stroke
-			(width 0)
-			(type default)
-		)
-	)
-	(wire
-		(pts
-			(xy 96.52 91.44) (xy 148.59 91.44)
-		)
-		(stroke
-			(width 0)
-			(type default)
-		)
-	)
-	(wire
-		(pts
-			(xy 97.79 27.94) (xy 127 27.94)
-		)
-		(stroke
-			(width 0)
-			(type default)
-		)
-	)
-	(wire
-		(pts
-			(xy 149.86 76.2) (xy 170.18 76.2)
-		)
-		(stroke
-			(width 0)
-			(type default)
-		)
-	)
-	(wire
-		(pts
-			(xy 46.99 74.93) (xy 99.06 74.93)
-		)
-		(stroke
-			(width 0)
-			(type default)
-		)
-	)
-	(wire
-		(pts
-			(xy 96.52 91.44) (xy 96.52 77.47)
-		)
-		(stroke
-			(width 0)
-			(type default)
-		)
-	)
-	(wire
-		(pts
-			(xy 170.18 54.61) (xy 191.77 54.61)
-		)
-		(stroke
-			(width 0)
-			(type default)
-		)
-	)
-	(wire
-		(pts
-			(xy 104.14 57.15) (xy 109.22 57.15)
 		)
 		(stroke
@@
 	)
 	(label "SWDCLK"
-		(at 46.99 74.93 0)
+		(at 46.99 72.39 0)
 		(effects
 			(font
@@
 		)
 	)
-	(label "RF_MOSI"
+	(label "MCU_MOSI"
 		(at 162.56 62.23 180)
 		(effects
@@
 	)
 	(label "SWDIO"
-		(at 46.99 77.47 0)
+		(at 46.99 69.85 0)
 		(effects
 			(font
@@
 		)
 	)
-	(label "RF_NSS"
+	(label "MCU_NSS"
 		(at 162.56 54.61 180)
 		(effects
@@
 		)
 	)
-	(label "RF_MISO"
+	(label "MCU_MISO"
 		(at 162.56 59.69 180)
 		(effects
@@
 		)
 	)
-	(label "RF_SCK"
+	(label "MCU_SCK"
 		(at 162.56 57.15 180)
 		(effects
@@
 	(symbol
 		(lib_id "power:+3.3V")
-		(at 46.99 72.39 270)
+		(at 46.99 77.47 270)
 		(unit 1)
 		(body_style 1)
@@
 		(fields_autoplaced yes)
 		(property "Reference" "#PWR05"
-			(at 43.18 72.39 0)
+			(at 43.18 77.47 0)
 			(hide yes)
 			(show_name no)
@@
 		)
 		(property "Value" "+3.3V"
-			(at 50.8 72.3899 90)
+			(at 50.8 77.4699 90)
 			(show_name no)
 			(do_not_autoplace no)
@@
 		)
 		(property "Footprint" ""
-			(at 46.99 72.39 0)
+			(at 46.99 77.47 0)
 			(hide yes)
 			(show_name no)
@@
 		)
 		(property "Datasheet" ""
-			(at 46.99 72.39 0)
+			(at 46.99 77.47 0)
 			(hide yes)
 			(show_name no)
@@
 		)
 		(property "Description" "Power symbol creates a global label with name \"+3.3V\""
-			(at 46.99 72.39 0)
+			(at 46.99 77.47 0)
 			(hide yes)
 			(show_name no)
@@
 	(symbol
 		(lib_id "power:GND")
-		(at 46.99 69.85 90)
+		(at 46.99 74.93 90)
 		(unit 1)
 		(body_style 1)
@@
 		(fields_autoplaced yes)
 		(property "Reference" "#PWR04"
-			(at 53.34 69.85 0)
+			(at 53.34 74.93 0)
 			(hide yes)
 			(show_name no)
@@
 		)
 		(property "Value" "GND"
-			(at 50.8 69.8499 90)
+			(at 50.8 74.9299 90)
 			(show_name no)
 			(do_not_autoplace no)
@@
 		)
 		(property "Footprint" ""
-			(at 46.99 69.85 0)
+			(at 46.99 74.93 0)
 			(hide yes)
 			(show_name no)
@@
 		)
 		(property "Datasheet" ""
-			(at 46.99 69.85 0)
+			(at 46.99 74.93 0)
 			(hide yes)
 			(show_name no)
@@
 		)
 		(property "Description" "Power symbol creates a global label with name \"GND\" , ground"
-			(at 46.99 69.85 0)
+			(at 46.99 74.93 0)
 			(hide yes)
 			(show_name no)
@@
 			)
 		)
-		(property "Footprint" "Resistor_SMD:R_0402_1005Metric_Pad0.72x0.64mm_HandSolder"
+		(property "Footprint" "Resistor_SMD:R_0603_1608Metric_Pad0.98x0.95mm_HandSolder"
 			(at 85.852 116.84 90)
 			(hide yes)

Commit message: rrev 4
Parts:
- C2, C4: value 100n -> 100nF
- C3: value 10u -> 10uF
- D1: value STATUS -> KT-0603R
- J1: value Conn_01x05_Pin -> (none); footprint Connector_PinHeader_1.00mm:PinHeader_1x05_P1.00mm_Vertical -> Connector_PinHeader_2.54mm:PinHeader_1x05_P2.54mm_Vertical
- J2: value Conn_01x02_Pin -> (none); footprint Connector_PinHeader_1.00mm:PinHeader_1x02_P1.00mm_Vertical -> Connector_PinHeader_2.54mm:PinHeader_1x02_P2.54mm_Vertical
- R3: footprint Resistor_SMD:R_0603_1608Metric_Pad0.98x0.95mm_HandSolder -> Resistor_SMD:R_0402_1005Metric_Pad0.72x0.64mm_HandSolder
- R4: value 10k? -> 10k
- SW1: value SW_SPST -> TS-1088-AR02016; footprint UnEasy-LCSC:KEY-SMD_L3.9-W3.0-LS5.0-EH -> UnEasy-LCSC:SW-SMD_L3.9-W3.0-P4.45
- U2: value STM32C011F6Px -> STM32C051F8P6
Changed lines of the file:
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@@
 			)
 		)
-		(property "Value" "Conn_01x05_Pin"
+		(property "Value" ""
 			(at 42.545 67.31 0)
 			(show_name no)
@@
 			)
 		)
-		(property "Footprint" "Connector_PinHeader_1.00mm:PinHeader_1x05_P1.00mm_Vertical"
+		(property "Footprint" "Connector_PinHeader_2.54mm:PinHeader_1x05_P2.54mm_Vertical"
 			(at 41.91 74.93 0)
 			(hide yes)
@@
 			)
 		)
-		(property "Value" "STM32C011F6Px"
+		(property "Value" "STM32C051F8P6"
 			(at 129.1433 36.83 0)
 			(show_name no)
@@
 			)
 		)
-		(property "Value" "100n"
+		(property "Value" "100nF"
 			(at 114.3 33.0199 0)
 			(show_name no)
@@
 			)
 		)
-		(property "Value" "10k?"
+		(property "Value" "10k"
 			(at 91.44 46.9901 0)
 			(show_name no)
@@
 			)
 		)
-		(property "Value" "100n"
+		(property "Value" "100nF"
 			(at 82.55 49.5299 0)
 			(show_name no)
@@
 			)
 		)
-		(property "Value" "SW_SPST"
+		(property "Value" "TS-1088-AR02016"
 			(at 59.436 50.8 90)
 			(show_name no)
@@
 			)
 		)
-		(property "Footprint" "UnEasy-LCSC:KEY-SMD_L3.9-W3.0-LS5.0-EH"
+		(property "Footprint" "UnEasy-LCSC:SW-SMD_L3.9-W3.0-P4.45"
 			(at 69.85 49.53 0)
 			(hide yes)
@@
 			)
 		)
-		(property "Value" "Conn_01x02_Pin"
+		(property "Value" ""
 			(at 211.455 64.77 0)
 			(show_name no)
@@
 			)
 		)
-		(property "Footprint" "Connector_PinHeader_1.00mm:PinHeader_1x02_P1.00mm_Vertical"
+		(property "Footprint" "Connector_PinHeader_2.54mm:PinHeader_1x02_P2.54mm_Vertical"
 			(at 212.09 67.31 0)
 			(hide yes)
@@
 			)
 		)
-		(property "Value" "10u"
+		(property "Value" "10uF"
 			(at 101.6 33.0199 0)
 			(show_name no)
@@
 			)
 		)
-		(property "Value" "STATUS"
+		(property "Value" "KT-0603R"
 			(at 182.88 81.788 0)
 			(show_name no)
@@
 			)
 		)
-		(property "Footprint" "Resistor_SMD:R_0603_1608Metric_Pad0.98x0.95mm_HandSolder"
+		(property "Footprint" "Resistor_SMD:R_0402_1005Metric_Pad0.72x0.64mm_HandSolder"
 			(at 85.852 116.84 90)
 			(hide yes)

Commit message: Revert "rrev 4"
Parts:
- C2, C4: value 100nF -> 100n
- C3: value 10uF -> 10u
- D1: value KT-0603R -> STATUS
- J1: value (none) -> Conn_01x05_Pin; footprint Connector_PinHeader_2.54mm:PinHeader_1x05_P2.54mm_Vertical -> Connector_PinHeader_1.00mm:PinHeader_1x05_P1.00mm_Vertical
- J2: value (none) -> Conn_01x02_Pin; footprint Connector_PinHeader_2.54mm:PinHeader_1x02_P2.54mm_Vertical -> Connector_PinHeader_1.00mm:PinHeader_1x02_P1.00mm_Vertical
- R3: footprint Resistor_SMD:R_0402_1005Metric_Pad0.72x0.64mm_HandSolder -> Resistor_SMD:R_0603_1608Metric_Pad0.98x0.95mm_HandSolder
- R4: value 10k -> 10k?
- SW1: value TS-1088-AR02016 -> SW_SPST; footprint UnEasy-LCSC:SW-SMD_L3.9-W3.0-P4.45 -> UnEasy-LCSC:KEY-SMD_L3.9-W3.0-LS5.0-EH
- U2: value STM32C051F8P6 -> STM32C011F6Px
Changed lines of the file:
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@@
 			)
 		)
-		(property "Value" ""
+		(property "Value" "Conn_01x05_Pin"
 			(at 42.545 67.31 0)
 			(show_name no)
@@
 			)
 		)
-		(property "Footprint" "Connector_PinHeader_2.54mm:PinHeader_1x05_P2.54mm_Vertical"
+		(property "Footprint" "Connector_PinHeader_1.00mm:PinHeader_1x05_P1.00mm_Vertical"
 			(at 41.91 74.93 0)
 			(hide yes)
@@
 			)
 		)
-		(property "Value" "STM32C051F8P6"
+		(property "Value" "STM32C011F6Px"
 			(at 129.1433 36.83 0)
 			(show_name no)
@@
 			)
 		)
-		(property "Value" "100nF"
+		(property "Value" "100n"
 			(at 114.3 33.0199 0)
 			(show_name no)
@@
 			)
 		)
-		(property "Value" "10k"
+		(property "Value" "10k?"
 			(at 91.44 46.9901 0)
 			(show_name no)
@@
 			)
 		)
-		(property "Value" "100nF"
+		(property "Value" "100n"
 			(at 82.55 49.5299 0)
 			(show_name no)
@@
 			)
 		)
-		(property "Value" "TS-1088-AR02016"
+		(property "Value" "SW_SPST"
 			(at 59.436 50.8 90)
 			(show_name no)
@@
 			)
 		)
-		(property "Footprint" "UnEasy-LCSC:SW-SMD_L3.9-W3.0-P4.45"
+		(property "Footprint" "UnEasy-LCSC:KEY-SMD_L3.9-W3.0-LS5.0-EH"
 			(at 69.85 49.53 0)
 			(hide yes)
@@
 			)
 		)
-		(property "Value" ""
+		(property "Value" "Conn_01x02_Pin"
 			(at 211.455 64.77 0)
 			(show_name no)
@@
 			)
 		)
-		(property "Footprint" "Connector_PinHeader_2.54mm:PinHeader_1x02_P2.54mm_Vertical"
+		(property "Footprint" "Connector_PinHeader_1.00mm:PinHeader_1x02_P1.00mm_Vertical"
 			(at 212.09 67.31 0)
 			(hide yes)
@@
 			)
 		)
-		(property "Value" "10uF"
+		(property "Value" "10u"
 			(at 101.6 33.0199 0)
 			(show_name no)
@@
 			)
 		)
-		(property "Value" "KT-0603R"
+		(property "Value" "STATUS"
 			(at 182.88 81.788 0)
 			(show_name no)
@@
 			)
 		)
-		(property "Footprint" "Resistor_SMD:R_0402_1005Metric_Pad0.72x0.64mm_HandSolder"
+		(property "Footprint" "Resistor_SMD:R_0603_1608Metric_Pad0.98x0.95mm_HandSolder"
 			(at 85.852 116.84 90)
 			(hide yes)
