File: boards/field_device/mcu.kicad_sch (KiCad schematic)
At the start: 19 parts, among them SW1 TS-1088-AR02016, U2 STM32C051F8P6

Commit message: rev 5?
Parts:
- removed R12, R4: 10k, Resistor_SMD:R_0402_1005Metric_Pad0.72x0.64mm_HandSolder, symbol Device:R
- removed R5: 22R, Resistor_SMD:R_0402_1005Metric_Pad0.72x0.64mm_HandSolder, symbol Device:R
- C2: value 100nF -> 100n
- renumbered R11 to R10, R6 to R5, R7 to R6, R8 to R7, R9 to R8, R10 to R9
Connections:
- net MCU_NSS is gone; now on net RF_NSS: U2.11 (PA4)
- net +3.3V: no longer R2.2, R3.2
- net I2C_BUS_PWR: now reaches U2.7 (PA0)
- net I2C_BUS_PWR: now also R2.2, R3.2
- no-connect marks 3 -> 2
Other:
- title: (none) -> Field Device MCU

Commit message: change components to fit manufacturing capability
Parts:
- C2: value 100n -> 100nF
Changed lines of the file:
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@@
 			)
 		)
-		(property "Value" "100n"
+		(property "Value" "100nF"
 			(at 82.55 49.5299 0)
 			(show_name no)

Commit message: idk atp
Parts:
- C2, C4: value 100nF -> CL05B104KO5NNNC 100nF
- C3: value 10uF -> CL10A106KP8NNNC 10uF
- R10, R2, R3: value 10k -> 0402WGF1002TCE 10k
- R5, R6, R7: value 22R -> 0402WGF220JTCE 22R
Changed lines of the file:
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@@
 			)
 		)
-		(property "Value" "22R"
+		(property "Value" "0402WGF220JTCE 22R"
 			(at 186.944 59.69 90)
 			(show_name no)
@@
 			)
 		)
-		(property "Value" "10k"
+		(property "Value" "0402WGF1002TCE 10k"
 			(at 80.01 118.1099 0)
 			(show_name no)
@@
 			)
 		)
-		(property "Value" "100nF"
+		(property "Value" "CL05B104KO5NNNC 100nF"
 			(at 114.3 33.0199 0)
 			(show_name no)
@@
 			)
 		)
-		(property "Value" "22R"
+		(property "Value" "0402WGF220JTCE 22R"
 			(at 186.944 57.15 90)
 			(show_name no)
@@
 			)
 		)
-		(property "Value" "22R"
+		(property "Value" "0402WGF220JTCE 22R"
 			(at 186.944 62.23 90)
 			(show_name no)
@@
 			)
 		)
-		(property "Value" "100nF"
+		(property "Value" "CL05B104KO5NNNC 100nF"
 			(at 82.55 49.5299 0)
 			(show_name no)
@@
 			)
 		)
-		(property "Value" "10uF"
+		(property "Value" "CL10A106KP8NNNC 10uF"
 			(at 101.6 33.0199 0)
 			(show_name no)
@@
 			)
 		)
-		(property "Value" "10k"
+		(property "Value" "0402WGF1002TCE 10k"
 			(at 90.17 118.1099 0)
 			(show_name no)
@@
 			)
 		)
-		(property "Value" "10k"
+		(property "Value" "0402WGF1002TCE 10k"
 			(at 173.99 81.788 90)
 			(show_name no)
